File: vr_module.sch (KiCad schematic (older format))
At the start: 26 parts, among them J1 Conn_01x07, U1 LM393, U2 NC7SB3157P6X, U3 74HC00, U4 NC7SB3157P6X, U5 SRV05-4, U6 MCP6004

Commit message: add power caps, silk on bottom
Parts:
- added C6: 10n, Capacitor_SMD:C_0603_1608Metric, symbol Device:C
- added C7: 1u, Capacitor_SMD:C_0603_1608Metric, symbol Device:C
Connections:
- net +5V: now also C6.1, C7.1
- net GND: now also C6.2, C7.2
Other:
- note added: "Differential to single ended conversion"
- note added: "RS Latch\nTracks which edge happened last"
- moved on the sheet: U3A, U3B
Changed lines of the file:
@@
 $EndComp
 Wire Wire Line
-	7150 2450 7550 2450
+	7150 2450 7650 2450
 Connection ~ 7150 2450
 Wire Wire Line
-	7150 3100 7550 3100
+	7150 3100 7650 3100
 Connection ~ 7150 3100
 Wire Wire Line
-	7550 2650 7500 2650
-Wire Wire Line
-	7500 2650 7500 2750
-Wire Wire Line
-	7500 2750 8200 2850
-Wire Wire Line
-	8200 2850 8200 3000
-Wire Wire Line
-	8200 3000 8150 3000
-Wire Wire Line
-	7550 2900 7500 2900
-Wire Wire Line
-	7500 2900 7500 2800
-Wire Wire Line
-	7500 2800 8200 2700
-Wire Wire Line
-	8200 2700 8200 2550
-Wire Wire Line
-	8200 2550 8150 2550
+	7650 2650 7600 2650
+Wire Wire Line
+	7600 2650 7600 2750
+Wire Wire Line
+	7600 2750 8300 2850
+Wire Wire Line
+	8300 2850 8300 3000
+Wire Wire Line
+	8300 3000 8250 3000
+Wire Wire Line
+	7650 2900 7600 2900
+Wire Wire Line
+	7600 2900 7600 2800
+Wire Wire Line
+	7600 2800 8300 2700
+Wire Wire Line
+	8300 2700 8300 2550
+Wire Wire Line
+	8300 2550 8250 2550
 $Comp
 L power:GND #PWR0103
@@
 L 74xx:74HC00 U3
 U 1 1 5FF97A18
-P 7850 2550
-F 0 "U3" H 7850 2550 50  0000 C CNN
-F 1 "74HC00" H 7850 2784 50  0001 C CNN
-F 2 "Package_SO:SOIC-14_3.9x8.7mm_P1.27mm" H 7850 2550 50  0001 C CNN
-F 3 "http://www.ti.com/lit/gpn/sn74hc00" H 7850 2550 50  0001 C CNN
-F 4 "C5586" H 7850 2550 50  0001 C CNN "LCSC"
-	1    7850 2550
+P 7950 2550
+F 0 "U3" H 7950 2550 50  0000 C CNN
+F 1 "74HC00" H 7950 2784 50  0001 C CNN
+F 2 "Package_SO:SOIC-14_3.9x8.7mm_P1.27mm" H 7950 2550 50  0001 C CNN
+F 3 "http://www.ti.com/lit/gpn/sn74hc00" H 7950 2550 50  0001 C CNN
+F 4 "C5586" H 7950 2550 50  0001 C CNN "LCSC"
+	1    7950 2550
 	1    0    0    -1
 $EndComp
@@
 L 74xx:74HC00 U3
 U 2 1 5FF9999F
-P 7850 3000
-F 0 "U3" H 7850 3000 50  0000 C CNN
-F 1 "74HC00" H 7850 2750 50  0001 C CNN
-F 2 "Package_SO:SOIC-14_3.9x8.7mm_P1.27mm" H 7850 3000 50  0001 C CNN
-F 3 "http://www.ti.com/lit/gpn/sn74hc00" H 7850 3000 50  0001 C CNN
-F 4 "C5586" H 7850 3000 50  0001 C CNN "LCSC"
-	2    7850 3000
+P 7950 3000
+F 0 "U3" H 7950 3000 50  0000 C CNN
+F 1 "74HC00" H 7950 2750 50  0001 C CNN
+F 2 "Package_SO:SOIC-14_3.9x8.7mm_P1.27mm" H 7950 3000 50  0001 C CNN
+F 3 "http://www.ti.com/lit/gpn/sn74hc00" H 7950 3000 50  0001 C CNN
+F 4 "C5586" H 7950 3000 50  0001 C CNN "LCSC"
+	2    7950 3000
 	1    0    0    -1
 $EndComp
@@
 	6750 1600 6850 1600
 Wire Wire Line
-	8200 2550 8450 2550
-Connection ~ 8200 2550
+	8300 2550 8550 2550
+Connection ~ 8300 2550
 Wire Wire Line
 	5550 2750 4750 2750
@@
 	0    -1   -1   0
 $EndComp
-Text GLabel 8450 2550 2    50   Input ~ 0
+Text GLabel 8550 2550 2    50   Input ~ 0
 output
 Text GLabel 4600 5850 0    50   Input ~ 0
@@
 Text GLabel 4600 5950 0    50   Input ~ 0
 analog_out
+Wire Notes Line
+	5000 2050 3500 2050
+Wire Notes Line
+	3500 2050 3500 3650
+Wire Notes Line
+	3500 3650 5000 3650
+Wire Notes Line
+	5000 3650 5000 2050
+Text Notes 3500 2150 0    50   ~ 0
+Differential to single ended conversion
+Wire Notes Line
+	7550 3250 8900 3250
+Wire Notes Line
+	8900 2150 7550 2150
+Text Notes 7600 2350 0    50   ~ 0
+RS Latch\nTracks which edge happened last
+Wire Notes Line
+	8900 2150 8900 3250
+Wire Notes Line
+	7550 3250 7550 2150
+$Comp
+L power:+5V #PWR0122
+U 1 1 602BE586
+P 8200 1000
+F 0 "#PWR0122" H 8200 850 50  0001 C CNN
+F 1 "+5V" H 8215 1173 50  0000 C CNN
+F 2 "" H 8200 1000 50  0001 C CNN
+F 3 "" H 8200 1000 50  0001 C CNN
+	1    8200 1000
+	1    0    0    -1
+$EndComp
+$Comp
+L power:GND #PWR0123
+U 1 1 602BED94
+P 8200 1300
+F 0 "#PWR0123" H 8200 1050 50  0001 C CNN
+F 1 "GND" H 8205 1127 50  0000 C CNN
+F 2 "" H 8200 1300 50  0001 C CNN
+F 3 "" H 8200 1300 50  0001 C CNN
+	1    8200 1300
+	1    0    0    -1
+$EndComp
+$Comp
+L Device:C C6
+U 1 1 602BF9F0
+P 8200 1150
+F 0 "C6" H 8315 1196 50  0000 L CNN
+F 1 "10n" H 8315 1105 50  0000 L CNN
+F 2 "Capacitor_SMD:C_0603_1608Metric" H 8238 1000 50  0001 C CNN
+F 3 "~" H 8200 1150 50  0001 C CNN
+	1    8200 1150
+	1    0    0    -1
+$EndComp
+$Comp
+L power:+5V #PWR0124
+U 1 1 602D4C21
+P 8600 1000
+F 0 "#PWR0124" H 8600 850 50  0001 C CNN
+F 1 "+5V" H 8615 1173 50  0000 C CNN
+F 2 "" H 8600 1000 50  0001 C CNN
+F 3 "" H 8600 1000 50  0001 C CNN
+	1    8600 1000
+	1    0    0    -1
+$EndComp
+$Comp
+L power:GND #PWR0125
+U 1 1 602D4C27
+P 8600 1300
+F 0 "#PWR0125" H 8600 1050 50  0001 C CNN
+F 1 "GND" H 8605 1127 50  0000 C CNN
+F 2 "" H 8600 1300 50  0001 C CNN
+F 3 "" H 8600 1300 50  0001 C CNN
+	1    8600 1300
+	1    0    0    -1
+$EndComp
+$Comp
+L Device:C C7
+U 1 1 602D4C2D
+P 8600 1150
+F 0 "C7" H 8715 1241 50  0000 L CNN
+F 1 "1u" H 8715 1150 50  0000 L CNN
+F 2 "Capacitor_SMD:C_0603_1608Metric" H 8715 1059 50  0000 L CNN
+F 3 "~" H 8600 1150 50  0001 C CNN
+	1    8600 1150
+	1    0    0    -1
+$EndComp
 $EndSCHEMATC

Commit message: filter pwm harder
Parts:
- added C?: 470n, Capacitor_SMD:C_0402_1005Metric, symbol Device:C
- added R?: 10k, Resistor_SMD:R_0402_1005Metric, symbol Device:R
- R12: value 33k -> 68k
Connections:
- net GND: now also C?.2
- net thresh_input: now also R?.1; no longer R11.1
- new net: C?.1, R11.1, R?.2
Other:
- moved on the sheet: C3, R11, R12, R13, R14, U6C, U6D
Changed lines of the file:
@@
 L Amplifier_Operational:MCP6004 U6
 U 3 1 60039068
-P 8400 5650
-F 0 "U6" H 8400 5650 50  0000 C CNN
-F 1 "MCP6004" H 8400 5926 50  0001 C CNN
-F 2 "Package_SO:TSSOP-14_4.4x5mm_P0.65mm" H 8350 5750 50  0001 C CNN
-F 3 "http://ww1.microchip.com/downloads/en/DeviceDoc/21733j.pdf" H 8450 5850 50  0001 C CNN
-F 4 "C50282" H 8400 5650 50  0001 C CNN "LCSC"
-	3    8400 5650
+P 8600 5800
+F 0 "U6" H 8600 5800 50  0000 C CNN
+F 1 "MCP6004" H 8600 6076 50  0001 C CNN
+F 2 "Package_SO:TSSOP-14_4.4x5mm_P0.65mm" H 8550 5900 50  0001 C CNN
+F 3 "http://ww1.microchip.com/downloads/en/DeviceDoc/21733j.pdf" H 8650 6000 50  0001 C CNN
+F 4 "C50282" H 8600 5800 50  0001 C CNN "LCSC"
+	3    8600 5800
 	1    0    0    -1
 $EndComp
@@
 L Amplifier_Operational:MCP6004 U6
 U 4 1 60039EA7
-P 9950 6050
-F 0 "U6" H 9950 6050 50  0000 C CNN
-F 1 "MCP6004" H 9950 6326 50  0001 C CNN
-F 2 "Package_SO:TSSOP-14_4.4x5mm_P0.65mm" H 9900 6150 50  0001 C CNN
-F 3 "http://ww1.microchip.com/downloads/en/DeviceDoc/21733j.pdf" H 10000 6250 50  0001 C CNN
-F 4 "C50282" H 9950 6050 50  0001 C CNN "LCSC"
-	4    9950 6050
+P 10150 6200
+F 0 "U6" H 10150 6200 50  0000 C CNN
+F 1 "MCP6004" H 10150 6476 50  0001 C CNN
+F 2 "Package_SO:TSSOP-14_4.4x5mm_P0.65mm" H 10100 6300 50  0001 C CNN
+F 3 "http://ww1.microchip.com/downloads/en/DeviceDoc/21733j.pdf" H 10200 6400 50  0001 C CNN
+F 4 "C50282" H 10150 6200 50  0001 C CNN "LCSC"
+	4    10150 6200
 	1    0    0    1
 $EndComp
@@
 L Device:R R11
 U 1 1 600DE66A
-P 7450 5300
-F 0 "R11" H 7520 5346 50  0000 L CNN
-F 1 "10k" H 7520 5255 50  0000 L CNN
-F 2 "Resistor_SMD:R_0402_1005Metric" V 7380 5300 50  0001 C CNN
-F 3 "~" H 7450 5300 50  0001 C CNN
-	1    7450 5300
+P 7650 5450
+F 0 "R11" H 7720 5496 50  0000 L CNN
+F 1 "10k" H 7720 5405 50  0000 L CNN
+F 2 "Resistor_SMD:R_0402_1005Metric" V 7580 5450 50  0001 C CNN
+F 3 "~" H 7650 5450 50  0001 C CNN
+	1    7650 5450
 	1    0    0    -1
 $EndComp
@@
 L Device:R R12
 U 1 1 600DF2EE
-P 7450 5800
-F 0 "R12" H 7520 5846 50  0000 L CNN
-F 1 "33k" H 7520 5755 50  0000 L CNN
-F 2 "Resistor_SMD:R_0402_1005Metric" V 7380 5800 50  0001 C CNN
-F 3 "~" H 7450 5800 50  0001 C CNN
-	1    7450 5800
+P 7650 5950
+F 0 "R12" H 7720 5996 50  0000 L CNN
+F 1 "68k" H 7720 5905 50  0000 L CNN
+F 2 "Resistor_SMD:R_0402_1005Metric" V 7580 5950 50  0001 C CNN
+F 3 "~" H 7650 5950 50  0001 C CNN
+	1    7650 5950
 	1    0    0    -1
 $EndComp
@@
 L power:GND #PWR0115
 U 1 1 600E258B
-P 7450 5950
-F 0 "#PWR0115" H 7450 5700 50  0001 C CNN
-F 1 "GND" H 7455 5777 50  0001 C CNN
-F 2 "" H 7450 5950 50  0001 C CNN
-F 3 "" H 7450 5950 50  0001 C CNN
-	1    7450 5950
+P 7650 6100
+F 0 "#PWR0115" H 7650 5850 50  0001 C CNN
+F 1 "GND" H 7655 5927 50  0001 C CNN
+F 2 "" H 7650 6100 50  0001 C CNN
+F 3 "" H 7650 6100 50  0001 C CNN
+	1    7650 6100
 	-1   0    0    -1
 $EndComp
 Wire Wire Line
-	8100 5750 8000 5750
-Wire Wire Line
-	8000 5750 8000 6000
-Wire Wire Line
-	8000 6000 8800 6000
-Wire Wire Line
-	8800 6000 8800 5650
-Wire Wire Line
-	8800 5650 8700 5650
-Wire Wire Line
-	8100 5550 7450 5550
-Wire Wire Line
-	7450 5550 7450 5450
-Wire Wire Line
-	7450 5550 7450 5650
-Connection ~ 7450 5550
+	8300 5900 8200 5900
+Wire Wire Line
+	8200 5900 8200 6150
+Wire Wire Line
+	8200 6150 9000 6150
+Wire Wire Line
+	9000 6150 9000 5800
+Wire Wire Line
+	9000 5800 8900 5800
+Wire Wire Line
+	8300 5700 7650 5700
+Wire Wire Line
+	7650 5700 7650 5600
+Wire Wire Line
+	7650 5700 7650 5800
+Connection ~ 7650 5700
 $Comp
 L Device:R R13
 U 1 1 600F5040
-P 9300 5650
-F 0 "R13" V 9093 5650 50  0000 C CNN
-F 1 "10k" V 9184 5650 50  0000 C CNN
-F 2 "Resistor_SMD:R_0402_1005Metric" V 9230 5650 50  0001 C CNN
-F 3 "~" H 9300 5650 50  0001 C CNN
-	1    9300 5650
+P 9500 5800
+F 0 "R13" V 9293 5800 50  0000 C CNN
+F 1 "10k" V 9384 5800 50  0000 C CNN
+F 2 "Resistor_SMD:R_0402_1005Metric" V 9430 5800 50  0001 C CNN
+F 3 "~" H 9500 5800 50  0001 C CNN
+	1    9500 5800
 	0    1    1    0
 $EndComp
@@
 L Device:R R14
 U 1 1 600F8206
-P 9950 5650
-F 0 "R14" V 9743 5650 50  0000 C CNN
-F 1 "10k" V 9834 5650 50  0000 C CNN
-F 2 "Resistor_SMD:R_0402_1005Metric" V 9880 5650 50  0001 C CNN
-F 3 "~" H 9950 5650 50  0001 C CNN
-	1    9950 5650
+P 10150 5800
+F 0 "R14" V 9943 5800 50  0000 C CNN
+F 1 "10k" V 10034 5800 50  0000 C CNN
+F 2 "Resistor_SMD:R_0402_1005Metric" V 10080 5800 50  0001 C CNN
+F 3 "~" H 10150 5800 50  0001 C CNN
+	1    10150 5800
 	0    1    1    0
 $EndComp
 Wire Wire Line
-	9650 5950 9600 5950
-Wire Wire Line
-	9600 5950 9600 5650
-Wire Wire Line
-	9600 5650 9450 5650
-Wire Wire Line
-	9150 5650 8800 5650
-Connection ~ 8800 5650
-Wire Wire Line
-	9600 5650 9800 5650
-Connection ~ 9600 5650
-Wire Wire Line
-	10100 5650 10350 5650
-Wire Wire Line
-	10350 5650 10350 6050
-Wire Wire Line
-	10350 6050 10250 6050
-Text GLabel 9500 6150 0    50   Input ~ 0
+	9850 6100 9800 6100
+Wire Wire Line
+	9800 6100 9800 5800
+Wire Wire Line
+	9800 5800 9650 5800
+Wire Wire Line
+	9350 5800 9000 5800
+Connection ~ 9000 5800
+Wire Wire Line
+	9800 5800 10000 5800
+Connection ~ 9800 5800
+Wire Wire Line
+	10300 5800 10550 5800
+Wire Wire Line
+	10550 5800 10550 6200
+Wire Wire Line
+	10550 6200 10450 6200
+Text GLabel 9700 6300 0    50   Input ~ 0
 Vref
 Wire Wire Line
-	9500 6150 9650 6150
-Text GLabel 10450 6050 2    50   Input ~ 0
+	9700 6300 9850 6300
+Text GLabel 10650 6200 2    50   Input ~ 0
 thresh_high
 Wire Wire Line
-	10450 6050 10350 6050
-Connection ~ 10350 6050
-Text GLabel 8900 6000 2    50   Input ~ 0
+	10650 6200 10550 6200
+Connection ~ 10550 6200
+Text GLabel 9100 6150 2    50   Input ~ 0
 thresh_low
 Wire Wire Line
-	8900 6000 8800 6000
-Connection ~ 8800 6000
-Text GLabel 7300 5000 0    50   Input ~ 0
+	9100 6150 9000 6150
+Connection ~ 9000 6150
+Text GLabel 6400 5150 0    50   Input ~ 0
 thresh_input
 Wire Wire Line
-	7300 5000 7450 5000
-Wire Wire Line
-	7450 5000 7450 5150
+	7650 5150 7650 5300
 Text GLabel 10300 4350 2    50   Input ~ 0
 Vref
@@
 L Device:C C3
 U 1 1 6016BDE4
-P 7050 5800
-F 0 "C3" H 7165 5846 50  0000 L CNN
-F 1 "100n" H 7165 5755 50  0000 L CNN
-F 2 "Capacitor_SMD:C_0402_1005Metric" H 7088 5650 50  0001 C CNN
-F 3 "~" H 7050 5800 50  0001 C CNN
-	1    7050 5800
+P 7250 5950
+F 0 "C3" H 7365 5996 50  0000 L CNN
+F 1 "100n" H 7365 5905 50  0000 L CNN
+F 2 "Capacitor_SMD:C_0402_1005Metric" H 7288 5800 50  0001 C CNN
+F 3 "~" H 7250 5950 50  0001 C CNN
+	1    7250 5950
 	1    0    0    -1
 $EndComp
@@
 L power:GND #PWR0118
 U 1 1 6016CD38
-P 7050 5950
-F 0 "#PWR0118" H 7050 5700 50  0001 C CNN
-F 1 "GND" H 7055 5777 50  0001 C CNN
-F 2 "" H 7050 5950 50  0001 C CNN
-F 3 "" H 7050 5950 50  0001 C CNN
-	1    7050 5950
+P 7250 6100
+F 0 "#PWR0118" H 7250 5850 50  0001 C CNN
+F 1 "GND" H 7255 5927 50  0001 C CNN
+F 2 "" H 7250 6100 50  0001 C CNN
+F 3 "" H 7250 6100 50  0001 C CNN
+	1    7250 6100
 	-1   0    0    -1
 $EndComp
 Wire Wire Line
-	7050 5650 7050 5550
-Wire Wire Line
-	7050 5550 7450 5550
+	7250 5800 7250 5700
+Wire Wire Line
+	7250 5700 7650 5700
 $Comp
 L Device:C C4
@@
 	1    0    0    -1
 $EndComp
+$Comp
+L Device:R R?
+U 1 1 602F8C0D
+P 6650 5150
+F 0 "R?" V 6443 5150 50  0000 C CNN
+F 1 "10k" V 6534 5150 50  0000 C CNN
+F 2 "Resistor_SMD:R_0402_1005Metric" V 6580 5150 50  0001 C CNN
+F 3 "~" H 6650 5150 50  0001 C CNN
+	1    6650 5150
+	0    -1   1    0
+$EndComp
+$Comp
+L Device:C C?
+U 1 1 602FA660
+P 6900 5400
+F 0 "C?" H 7015 5446 50  0000 L CNN
+F 1 "470n" H 7015 5355 50  0000 L CNN
+F 2 "Capacitor_SMD:C_0402_1005Metric" H 6938 5250 50  0001 C CNN
+F 3 "~" H 6900 5400 50  0001 C CNN
+	1    6900 5400
+	1    0    0    -1
+$EndComp
+$Comp
+L power:GND #PWR?
+U 1 1 602FACD3
+P 6900 5550
+F 0 "#PWR?" H 6900 5300 50  0001 C CNN
+F 1 "GND" H 6905 5377 50  0001 C CNN
+F 2 "" H 6900 5550 50  0001 C CNN
+F 3 "" H 6900 5550 50  0001 C CNN
+	1    6900 5550
+	-1   0    0    -1
+$EndComp
+Wire Wire Line
+	6800 5150 6900 5150
+Wire Wire Line
+	6900 5150 6900 5250
+Wire Wire Line
+	6500 5150 6400 5150
+Wire Wire Line
+	6900 5150 7650 5150
+Connection ~ 6900 5150
 $EndSCHEMATC

Commit message: lcsc numbers, optimize divider
Parts:
- C1, C2: LCSC (none) -> C15195
- C3, C4: LCSC (none) -> C1525
- C5: LCSC (none) -> C1523
- C6: footprint Capacitor_SMD:C_0603_1608Metric -> Capacitor_SMD:C_0402_1005Metric; LCSC (none) -> C15195
- C7: LCSC (none) -> C15849
- C8: renamed from C?; LCSC (none) -> C47339
- R1, R2: LCSC (none) -> C11702
- R10, R11, R13, R14, R9: LCSC (none) -> C25744
- R12: LCSC (none) -> C36871
- R15: renamed from R?; value 10k -> 12k; LCSC (none) -> C25752
- R3, R4, R5, R6: LCSC (none) -> C25741
- R7, R8: LCSC (none) -> C17414
Changed lines of the file:
@@
 F 2 "Capacitor_SMD:C_0402_1005Metric" H 6838 2300 50  0001 C CNN
 F 3 "~" H 6800 2450 50  0001 C CNN
+F 4 "C15195" H 6800 2450 50  0001 C CNN "LCSC"
 	1    6800 2450
 	0    1    1    0
@@
 F 2 "Resistor_SMD:R_0402_1005Metric" V 7080 2150 50  0001 C CNN
 F 3 "~" H 7150 2150 50  0001 C CNN
+F 4 "C11702" H 7150 2150 50  0001 C CNN "LCSC"
 	1    7150 2150
 	1    0    0    -1
@@
 F 2 "Capacitor_SMD:C_0402_1005Metric" H 6838 2950 50  0001 C CNN
 F 3 "~" H 6800 3100 50  0001 C CNN
+F 4 "C15195" H 6800 3100 50  0001 C CNN "LCSC"
 	1    6800 3100
 	0    1    -1   0
@@
 F 2 "Resistor_SMD:R_0402_1005Metric" V 7080 3400 50  0001 C CNN
 F 3 "~" H 7150 3400 50  0001 C CNN
+F 4 "C11702" H 7150 3400 50  0001 C CNN "LCSC"
 	1    7150 3400
 	1    0    0    1
@@
 F 2 "Resistor_SMD:R_0402_1005Metric" V 4280 2350 50  0001 C CNN
 F 3 "~" H 4350 2350 50  0001 C CNN
+F 4 "C25741" H 4350 2350 50  0001 C CNN "LCSC"
 	1    4350 2350
 	0    1    1    0
@@
 F 2 "Resistor_SMD:R_0402_1005Metric" V 3880 3250 50  0001 C CNN
 F 3 "~" H 3950 3250 50  0001 C CNN
+F 4 "C25741" H 3950 3250 50  0001 C CNN "LCSC"
 	1    3950 3250
 	1    0    0    -1
@@
 F 2 "Resistor_SMD:R_0402_1005Metric" V 3630 2850 50  0001 C CNN
 F 3 "~" H 3700 2850 50  0001 C CNN
+F 4 "C25741" H 3700 2850 50  0001 C CNN "LCSC"
 	1    3700 2850
 	0    -1   -1   0
@@
 F 2 "Resistor_SMD:R_0402_1005Metric" V 3630 2650 50  0001 C CNN
 F 3 "~" H 3700 2650 50  0001 C CNN
+F 4 "C25741" H 3700 2650 50  0001 C CNN "LCSC"
 	1    3700 2650
 	0    1    1    0
@@
 F 2 "Resistor_SMD:R_0805_2012Metric" V 2130 2650 50  0001 C CNN
 F 3 "~" H 2200 2650 50  0001 C CNN
+F 4 "C17414" H 2200 2650 50  0001 C CNN "LCSC"
 	1    2200 2650
 	0    -1   -1   0
@@
 F 2 "Resistor_SMD:R_0805_2012Metric" V 2130 2850 50  0001 C CNN
 F 3 "~" H 2200 2850 50  0001 C CNN
+F 4 "C17414" H 2200 2850 50  0001 C CNN "LCSC"
 	1    2200 2850
 	0    1    1    0
@@
 F 2 "Resistor_SMD:R_0402_1005Metric" V 7580 5450 50  0001 C CNN
 F 3 "~" H 7650 5450 50  0001 C CNN
+F 4 "C25744" H 7650 5450 50  0001 C CNN "LCSC"
 	1    7650 5450
 	1    0    0    -1
@@
 F 2 "Resistor_SMD:R_0402_1005Metric" V 7580 5950 50  0001 C CNN
 F 3 "~" H 7650 5950 50  0001 C CNN
+F 4 "C36871" H 7650 5950 50  0001 C CNN "LCSC"
 	1    7650 5950
 	1    0    0    -1
@@
 F 2 "Resistor_SMD:R_0402_1005Metric" V 9430 5800 50  0001 C CNN
 F 3 "~" H 9500 5800 50  0001 C CNN
+F 4 "C25744" H 9500 5800 50  0001 C CNN "LCSC"
 	1    9500 5800
 	0    1    1    0
@@
 F 2 "Resistor_SMD:R_0402_1005Metric" V 10080 5800 50  0001 C CNN
 F 3 "~" H 10150 5800 50  0001 C CNN
+F 4 "C25744" H 10150 5800 50  0001 C CNN "LCSC"
 	1    10150 5800
 	0    1    1    0
@@
 F 2 "Resistor_SMD:R_0402_1005Metric" V 8980 4450 50  0001 C CNN
 F 3 "~" H 9050 4450 50  0001 C CNN
+F 4 "C25744" H 9050 4450 50  0001 C CNN "LCSC"
 	1    9050 4450
 	1    0    0    -1
@@
 F 2 "Resistor_SMD:R_0402_1005Metric" V 8980 4050 50  0001 C CNN
 F 3 "~" H 9050 4050 50  0001 C CNN
+F 4 "C25744" H 9050 4050 50  0001 C CNN "LCSC"
 	1    9050 4050
 	1    0    0    -1
@@
 F 2 "Capacitor_SMD:C_0402_1005Metric" H 7288 5800 50  0001 C CNN
 F 3 "~" H 7250 5950 50  0001 C CNN
+F 4 "C1525" H 7250 5950 50  0001 C CNN "LCSC"
 	1    7250 5950
 	1    0    0    -1
@@
 F 2 "Capacitor_SMD:C_0402_1005Metric" H 8688 4300 50  0001 C CNN
 F 3 "~" H 8650 4450 50  0001 C CNN
+F 4 "C1525" H 8650 4450 50  0001 C CNN "LCSC"
 	1    8650 4450
 	1    0    0    -1
@@
 F 2 "Capacitor_SMD:C_0402_1005Metric" H 2850 2750 50  0001 C CNN
 F 3 "~" H 2850 2750 50  0001 C CNN
+F 4 "C1523" H 2850 2750 50  0001 C CNN "LCSC"
 	1    2850 2750
 	1    0    0    -1
@@
 F 0 "C6" H 8315 1196 50  0000 L CNN
 F 1 "10n" H 8315 1105 50  0000 L CNN
-F 2 "Capacitor_SMD:C_0603_1608Metric" H 8238 1000 50  0001 C CNN
+F 2 "Capacitor_SMD:C_0402_1005Metric" H 8238 1000 50  0001 C CNN
 F 3 "~" H 8200 1150 50  0001 C CNN
+F 4 "C15195" H 8200 1150 50  0001 C CNN "LCSC"
 	1    8200 1150
 	1    0    0    -1
@@
 U 1 1 602D4C2D
 P 8600 1150
-F 0 "C7" H 8715 1241 50  0000 L CNN
-F 1 "1u" H 8715 1150 50  0000 L CNN
-F 2 "Capacitor_SMD:C_0603_1608Metric" H 8715 1059 50  0000 L CNN
+F 0 "C7" H 8715 1196 50  0000 L CNN
+F 1 "1u" H 8715 1105 50  0000 L CNN
+F 2 "Capacitor_SMD:C_0603_1608Metric" H 8715 1059 50  0001 L CNN
 F 3 "~" H 8600 1150 50  0001 C CNN
+F 4 "C15849" H 8600 1150 50  0001 C CNN "LCSC"
 	1    8600 1150
 	1    0    0    -1
 $EndComp
 $Comp
-L Device:R R?
+L Device:R R15
 U 1 1 602F8C0D
 P 6650 5150
-F 0 "R?" V 6443 5150 50  0000 C CNN
-F 1 "10k" V 6534 5150 50  0000 C CNN
+F 0 "R15" V 6443 5150 50  0000 C CNN
+F 1 "12k" V 6534 5150 50  0000 C CNN
 F 2 "Resistor_SMD:R_0402_1005Metric" V 6580 5150 50  0001 C CNN
 F 3 "~" H 6650 5150 50  0001 C CNN
+F 4 "C25752" H 6650 5150 50  0001 C CNN "LCSC"
 	1    6650 5150
 	0    -1   1    0
 $EndComp
 $Comp
-L Device:C C?
+L Device:C C8
 U 1 1 602FA660
 P 6900 5400
-F 0 "C?" H 7015 5446 50  0000 L CNN
+F 0 "C8" H 7015 5446 50  0000 L CNN
 F 1 "470n" H 7015 5355 50  0000 L CNN
 F 2 "Capacitor_SMD:C_0402_1005Metric" H 6938 5250 50  0001 C CNN
 F 3 "~" H 6900 5400 50  0001 C CNN
+F 4 "C47339" H 6900 5400 50  0001 C CNN "LCSC"
 	1    6900 5400
 	1    0    0    -1
 $EndComp
 $Comp
-L power:GND #PWR?
+L power:GND #PWR0126
 U 1 1 602FACD3
 P 6900 5550
-F 0 "#PWR?" H 6900 5300 50  0001 C CNN
+F 0 "#PWR0126" H 6900 5300 50  0001 C CNN
 F 1 "GND" H 6905 5377 50  0001 C CNN
 F 2 "" H 6900 5550 50  0001 C CNN

Commit message: add filter caps
Parts:
- added C10, C9: 10n, Capacitor_SMD:C_0402_1005Metric, symbol Device:C
Connections:
- net GND: now also C10.1, C9.1
- net at U1.2 (-), U2.4: now also C9.2
- net at U1.6 (_), U4.4: now also C10.2
Changed lines of the file:
@@
 	6150 1500 5550 1500
 Wire Wire Line
-	5550 1500 5550 2350
+	5550 1500 5550 1850
 Wire Wire Line
 	5550 2350 5700 2350
@@
 	6150 4050 5550 4050
 Wire Wire Line
-	5550 4050 5550 3200
+	5550 4050 5550 3750
 Wire Wire Line
 	5550 3200 5700 3200
@@
 	6900 5150 7650 5150
 Connection ~ 6900 5150
+$Comp
+L Device:C C9
+U 1 1 603744CE
+P 5800 1850
+F 0 "C9" V 5548 1850 50  0000 C CNN
+F 1 "10n" V 5639 1850 50  0000 C CNN
+F 2 "Capacitor_SMD:C_0402_1005Metric" H 5838 1700 50  0001 C CNN
+F 3 "~" H 5800 1850 50  0001 C CNN
+F 4 "C15195" H 5800 1850 50  0001 C CNN "LCSC"
+	1    5800 1850
+	0    1    1    0
+$EndComp
+$Comp
+L power:GND #PWR0127
+U 1 1 60375132
+P 5950 1850
+F 0 "#PWR0127" H 5950 1600 50  0001 C CNN
+F 1 "GND" H 5955 1677 50  0001 C CNN
+F 2 "" H 5950 1850 50  0001 C CNN
+F 3 "" H 5950 1850 50  0001 C CNN
+	1    5950 1850
+	0    -1   -1   0
+$EndComp
+Wire Wire Line
+	5650 1850 5550 1850
+Connection ~ 5550 1850
+Wire Wire Line
+	5550 1850 5550 2350
+$Comp
+L Device:C C10
+U 1 1 6038066A
+P 5800 3750
+F 0 "C10" V 5548 3750 50  0000 C CNN
+F 1 "10n" V 5639 3750 50  0000 C CNN
+F 2 "Capacitor_SMD:C_0402_1005Metric" H 5838 3600 50  0001 C CNN
+F 3 "~" H 5800 3750 50  0001 C CNN
+F 4 "C15195" H 5800 3750 50  0001 C CNN "LCSC"
+	1    5800 3750
+	0    1    1    0
+$EndComp
+$Comp
+L power:GND #PWR0128
+U 1 1 60380670
+P 5950 3750
+F 0 "#PWR0128" H 5950 3500 50  0001 C CNN
+F 1 "GND" H 5955 3577 50  0001 C CNN
+F 2 "" H 5950 3750 50  0001 C CNN
+F 3 "" H 5950 3750 50  0001 C CNN
+	1    5950 3750
+	0    -1   -1   0
+$EndComp
+Wire Wire Line
+	5650 3750 5550 3750
+Connection ~ 5550 3750
+Wire Wire Line
+	5550 3750 5550 3200
 $EndSCHEMATC
