File: vr_module.sch (KiCad schematic (older format))
At the start: 32 parts, among them J1 Conn_01x07, U1 LM393, U2 NC7SB3157P6X, U3 74HC00, U4 NC7SB3157P6X, U5 SRV05-4, U6 MCP6004

Commit message: drc
Connections:
- no-connect marks 0 -> 2
Changed lines of the file:
@@
 L power:GND #PWR0120
 U 1 1 601B40D4
-P 4600 5650
-F 0 "#PWR0120" H 4600 5400 50  0001 C CNN
-F 1 "GND" H 4605 5477 50  0001 C CNN
-F 2 "" H 4600 5650 50  0001 C CNN
-F 3 "" H 4600 5650 50  0001 C CNN
-	1    4600 5650
+P 4500 5650
+F 0 "#PWR0120" H 4500 5400 50  0001 C CNN
+F 1 "GND" H 4505 5477 50  0001 C CNN
+F 2 "" H 4500 5650 50  0001 C CNN
+F 3 "" H 4500 5650 50  0001 C CNN
+	1    4500 5650
 	0    1    -1   0
 $EndComp
@@
 L power:+5V #PWR0121
 U 1 1 601BBF3A
-P 4600 5750
-F 0 "#PWR0121" H 4600 5600 50  0001 C CNN
-F 1 "+5V" V 4615 5878 50  0000 L CNN
-F 2 "" H 4600 5750 50  0001 C CNN
-F 3 "" H 4600 5750 50  0001 C CNN
-	1    4600 5750
+P 4250 5750
+F 0 "#PWR0121" H 4250 5600 50  0001 C CNN
+F 1 "+5V" V 4265 5878 50  0000 L CNN
+F 2 "" H 4250 5750 50  0001 C CNN
+F 3 "" H 4250 5750 50  0001 C CNN
+	1    4250 5750
 	0    -1   -1   0
 $EndComp
@@
 Wire Wire Line
 	5550 3750 5550 3200
+Wire Wire Line
+	4250 5750 4300 5750
+$Comp
+L power:PWR_FLAG #FLG0101
+U 1 1 603A20E4
+P 4300 5750
+F 0 "#FLG0101" H 4300 5825 50  0001 C CNN
+F 1 "PWR_FLAG" H 4300 5923 50  0001 C CNN
+F 2 "" H 4300 5750 50  0001 C CNN
+F 3 "~" H 4300 5750 50  0001 C CNN
+	1    4300 5750
+	1    0    0    -1
+$EndComp
+Connection ~ 4300 5750
+Wire Wire Line
+	4300 5750 4600 5750
+Wire Wire Line
+	4500 5650 4550 5650
+$Comp
+L power:PWR_FLAG #FLG0102
+U 1 1 603AB746
+P 4550 5650
+F 0 "#FLG0102" H 4550 5725 50  0001 C CNN
+F 1 "PWR_FLAG" H 4550 5823 50  0001 C CNN
+F 2 "" H 4550 5650 50  0001 C CNN
+F 3 "~" H 4550 5650 50  0001 C CNN
+	1    4550 5650
+	1    0    0    -1
+$EndComp
+Connection ~ 4550 5650
+Wire Wire Line
+	4550 5650 4600 5650
+NoConn ~ 3550 1500
+NoConn ~ 3550 1700
 $EndSCHEMATC

Commit message: ground unused inputs to NAND
Parts:
- added unit 3 of U3
- added unit 4 of U3
Connections:
- net GND: now also U3.10, U3.12, U3.13, U3.9
Other:
- note added: "Unused gates"
- moved on the sheet: C4, R10, R9, U6B
Changed lines of the file:
@@
 L Amplifier_Operational:MCP6004 U6
 U 2 1 60037039
-P 9850 4350
-F 0 "U6" H 9850 4350 50  0000 C CNN
-F 1 "MCP6004" H 9850 4626 50  0001 C CNN
-F 2 "Package_SO:TSSOP-14_4.4x5mm_P0.65mm" H 9800 4450 50  0001 C CNN
-F 3 "http://ww1.microchip.com/downloads/en/DeviceDoc/21733j.pdf" H 9900 4550 50  0001 C CNN
-F 4 "C50282" H 9850 4350 50  0001 C CNN "LCSC"
-	2    9850 4350
+P 9000 4150
+F 0 "U6" H 9000 4150 50  0000 C CNN
+F 1 "MCP6004" H 9000 4426 50  0001 C CNN
+F 2 "Package_SO:TSSOP-14_4.4x5mm_P0.65mm" H 8950 4250 50  0001 C CNN
+F 3 "http://ww1.microchip.com/downloads/en/DeviceDoc/21733j.pdf" H 9050 4350 50  0001 C CNN
+F 4 "C50282" H 9000 4150 50  0001 C CNN "LCSC"
+	2    9000 4150
 	1    0    0    -1
 $EndComp
@@
 Wire Wire Line
 	7650 5150 7650 5300
-Text GLabel 10300 4350 2    50   Input ~ 0
+Text GLabel 9450 4150 2    50   Input ~ 0
 Vref
 Wire Wire Line
-	10300 4350 10200 4350
-Wire Wire Line
-	9550 4450 9450 4450
-Wire Wire Line
-	9450 4450 9450 4650
-Wire Wire Line
-	9450 4650 10200 4650
-Wire Wire Line
-	10200 4650 10200 4350
-Connection ~ 10200 4350
-Wire Wire Line
-	10200 4350 10150 4350
+	9450 4150 9350 4150
+Wire Wire Line
+	8700 4250 8600 4250
+Wire Wire Line
+	8600 4250 8600 4450
+Wire Wire Line
+	8600 4450 9350 4450
+Wire Wire Line
+	9350 4450 9350 4150
+Connection ~ 9350 4150
+Wire Wire Line
+	9350 4150 9300 4150
 $Comp
 L Device:R R10
 U 1 1 60151F59
-P 9050 4450
-F 0 "R10" H 9120 4496 50  0000 L CNN
-F 1 "10k" H 9120 4405 50  0000 L CNN
-F 2 "Resistor_SMD:R_0402_1005Metric" V 8980 4450 50  0001 C CNN
-F 3 "~" H 9050 4450 50  0001 C CNN
-F 4 "C25744" H 9050 4450 50  0001 C CNN "LCSC"
-	1    9050 4450
+P 8200 4250
+F 0 "R10" H 8270 4296 50  0000 L CNN
+F 1 "10k" H 8270 4205 50  0000 L CNN
+F 2 "Resistor_SMD:R_0402_1005Metric" V 8130 4250 50  0001 C CNN
+F 3 "~" H 8200 4250 50  0001 C CNN
+F 4 "C25744" H 8200 4250 50  0001 C CNN "LCSC"
+	1    8200 4250
 	1    0    0    -1
 $EndComp
@@
 L Device:R R9
 U 1 1 6015342D
-P 9050 4050
-F 0 "R9" H 9120 4096 50  0000 L CNN
-F 1 "10k" H 9120 4005 50  0000 L CNN
-F 2 "Resistor_SMD:R_0402_1005Metric" V 8980 4050 50  0001 C CNN
-F 3 "~" H 9050 4050 50  0001 C CNN
-F 4 "C25744" H 9050 4050 50  0001 C CNN "LCSC"
-	1    9050 4050
-	1    0    0    -1
-$EndComp
-Wire Wire Line
-	9550 4250 9050 4250
-Wire Wire Line
-	9050 4250 9050 4300
-Wire Wire Line
-	9050 4250 9050 4200
-Connection ~ 9050 4250
+P 8200 3850
+F 0 "R9" H 8270 3896 50  0000 L CNN
+F 1 "10k" H 8270 3805 50  0000 L CNN
+F 2 "Resistor_SMD:R_0402_1005Metric" V 8130 3850 50  0001 C CNN
+F 3 "~" H 8200 3850 50  0001 C CNN
+F 4 "C25744" H 8200 3850 50  0001 C CNN "LCSC"
+	1    8200 3850
+	1    0    0    -1
+$EndComp
+Wire Wire Line
+	8700 4050 8200 4050
+Wire Wire Line
+	8200 4050 8200 4100
+Wire Wire Line
+	8200 4050 8200 4000
+Connection ~ 8200 4050
 $Comp
 L power:GND #PWR0116
 U 1 1 6015A40F
-P 9050 4600
-F 0 "#PWR0116" H 9050 4350 50  0001 C CNN
-F 1 "GND" H 9055 4427 50  0000 C CNN
-F 2 "" H 9050 4600 50  0001 C CNN
-F 3 "" H 9050 4600 50  0001 C CNN
-	1    9050 4600
+P 8200 4400
+F 0 "#PWR0116" H 8200 4150 50  0001 C CNN
+F 1 "GND" H 8205 4227 50  0000 C CNN
+F 2 "" H 8200 4400 50  0001 C CNN
+F 3 "" H 8200 4400 50  0001 C CNN
+	1    8200 4400
 	1    0    0    -1
 $EndComp
@@
 L power:+5V #PWR0117
 U 1 1 6015AC84
-P 9050 3900
-F 0 "#PWR0117" H 9050 3750 50  0001 C CNN
-F 1 "+5V" H 9065 4073 50  0000 C CNN
-F 2 "" H 9050 3900 50  0001 C CNN
-F 3 "" H 9050 3900 50  0001 C CNN
-	1    9050 3900
+P 8200 3700
+F 0 "#PWR0117" H 8200 3550 50  0001 C CNN
+F 1 "+5V" H 8215 3873 50  0000 C CNN
+F 2 "" H 8200 3700 50  0001 C CNN
+F 3 "" H 8200 3700 50  0001 C CNN
+	1    8200 3700
 	1    0    0    -1
 $EndComp
@@
 L Device:C C4
 U 1 1 60172DAB
-P 8650 4450
-F 0 "C4" H 8765 4496 50  0000 L CNN
-F 1 "100n" H 8765 4405 50  0000 L CNN
-F 2 "Capacitor_SMD:C_0402_1005Metric" H 8688 4300 50  0001 C CNN
-F 3 "~" H 8650 4450 50  0001 C CNN
-F 4 "C1525" H 8650 4450 50  0001 C CNN "LCSC"
-	1    8650 4450
+P 7800 4250
+F 0 "C4" H 7915 4296 50  0000 L CNN
+F 1 "100n" H 7915 4205 50  0000 L CNN
+F 2 "Capacitor_SMD:C_0402_1005Metric" H 7838 4100 50  0001 C CNN
+F 3 "~" H 7800 4250 50  0001 C CNN
+F 4 "C1525" H 7800 4250 50  0001 C CNN "LCSC"
+	1    7800 4250
 	1    0    0    -1
 $EndComp
@@
 L power:GND #PWR0119
 U 1 1 601761B8
-P 8650 4600
-F 0 "#PWR0119" H 8650 4350 50  0001 C CNN
-F 1 "GND" H 8655 4427 50  0000 C CNN
-F 2 "" H 8650 4600 50  0001 C CNN
-F 3 "" H 8650 4600 50  0001 C CNN
-	1    8650 4600
-	1    0    0    -1
-$EndComp
-Wire Wire Line
-	8650 4300 8650 4250
-Wire Wire Line
-	8650 4250 9050 4250
+P 7800 4400
+F 0 "#PWR0119" H 7800 4150 50  0001 C CNN
+F 1 "GND" H 7805 4227 50  0000 C CNN
+F 2 "" H 7800 4400 50  0001 C CNN
+F 3 "" H 7800 4400 50  0001 C CNN
+	1    7800 4400
+	1    0    0    -1
+$EndComp
+Wire Wire Line
+	7800 4100 7800 4050
+Wire Wire Line
+	7800 4050 8200 4050
 $Comp
 L power:GND #PWR0120
@@
 NoConn ~ 3550 1500
 NoConn ~ 3550 1700
+$Comp
+L 74xx:74HC00 U3
+U 3 1 603F0D08
+P 10600 3950
+F 0 "U3" H 10600 3950 50  0000 C CNN
+F 1 "74HC00" H 10600 3700 50  0001 C CNN
+F 2 "Package_SO:SOIC-14_3.9x8.7mm_P1.27mm" H 10600 3950 50  0001 C CNN
+F 3 "http://www.ti.com/lit/gpn/sn74hc00" H 10600 3950 50  0001 C CNN
+F 4 "C5586" H 10600 3950 50  0001 C CNN "LCSC"
+	3    10600 3950
+	1    0    0    -1
+$EndComp
+$Comp
+L 74xx:74HC00 U3
+U 4 1 603F2881
+P 10600 4400
+F 0 "U3" H 10600 4400 50  0000 C CNN
+F 1 "74HC00" H 10600 4150 50  0001 C CNN
+F 2 "Package_SO:SOIC-14_3.9x8.7mm_P1.27mm" H 10600 4400 50  0001 C CNN
+F 3 "http://www.ti.com/lit/gpn/sn74hc00" H 10600 4400 50  0001 C CNN
+F 4 "C5586" H 10600 4400 50  0001 C CNN "LCSC"
+	4    10600 4400
+	1    0    0    -1
+$EndComp
+$Comp
+L power:GND #PWR01
+U 1 1 603F7133
+P 10300 3850
+F 0 "#PWR01" H 10300 3600 50  0001 C CNN
+F 1 "GND" H 10305 3677 50  0001 C CNN
+F 2 "" H 10300 3850 50  0001 C CNN
+F 3 "" H 10300 3850 50  0001 C CNN
+	1    10300 3850
+	0    1    -1   0
+$EndComp
+$Comp
+L power:GND #PWR02
+U 1 1 603F7FC4
+P 10300 4050
+F 0 "#PWR02" H 10300 3800 50  0001 C CNN
+F 1 "GND" H 10305 3877 50  0001 C CNN
+F 2 "" H 10300 4050 50  0001 C CNN
+F 3 "" H 10300 4050 50  0001 C CNN
+	1    10300 4050
+	0    1    -1   0
+$EndComp
+$Comp
+L power:GND #PWR03
+U 1 1 603F8380
+P 10300 4300
+F 0 "#PWR03" H 10300 4050 50  0001 C CNN
+F 1 "GND" H 10305 4127 50  0001 C CNN
+F 2 "" H 10300 4300 50  0001 C CNN
+F 3 "" H 10300 4300 50  0001 C CNN
+	1    10300 4300
+	0    1    -1   0
+$EndComp
+$Comp
+L power:GND #PWR04
+U 1 1 603F8770
+P 10300 4500
+F 0 "#PWR04" H 10300 4250 50  0001 C CNN
+F 1 "GND" H 10305 4327 50  0001 C CNN
+F 2 "" H 10300 4500 50  0001 C CNN
+F 3 "" H 10300 4500 50  0001 C CNN
+	1    10300 4500
+	0    1    -1   0
+$EndComp
+Wire Notes Line
+	10100 3600 10100 4650
+Wire Notes Line
+	10100 4650 11000 4650
+Wire Notes Line
+	11000 4650 11000 3600
+Wire Notes Line
+	11000 3600 10100 3600
+Text Notes 10200 3700 0    50   ~ 0
+Unused gates
 $EndSCHEMATC

Commit message: upgrade comparator
Parts:
- U1: value LM393 -> MAX9142; LCSC C7955 -> C18567
- U1: value LM393 -> MAX9142
Other:
- moved on the sheet: U2B, U4B
Changed lines of the file:
@@
 L power:GND #PWR0104
 U 1 1 5FF5AE6A
-P 10000 3100
-F 0 "#PWR0104" H 10000 2850 50  0001 C CNN
-F 1 "GND" H 10005 2927 50  0000 C CNN
-F 2 "" H 10000 3100 50  0001 C CNN
-F 3 "" H 10000 3100 50  0001 C CNN
-	1    10000 3100
+P 9350 3200
+F 0 "#PWR0104" H 9350 2950 50  0001 C CNN
+F 1 "GND" H 9355 3027 50  0000 C CNN
+F 2 "" H 9350 3200 50  0001 C CNN
+F 3 "" H 9350 3200 50  0001 C CNN
+	1    9350 3200
 	1    0    0    -1
 $EndComp
@@
 L power:GND #PWR0105
 U 1 1 5FF5B4BC
-P 11000 3100
-F 0 "#PWR0105" H 11000 2850 50  0001 C CNN
-F 1 "GND" H 11005 2927 50  0000 C CNN
-F 2 "" H 11000 3100 50  0001 C CNN
-F 3 "" H 11000 3100 50  0001 C CNN
-	1    11000 3100
+P 10350 3200
+F 0 "#PWR0105" H 10350 2950 50  0001 C CNN
+F 1 "GND" H 10355 3027 50  0000 C CNN
+F 2 "" H 10350 3200 50  0001 C CNN
+F 3 "" H 10350 3200 50  0001 C CNN
+	1    10350 3200
 	1    0    0    -1
 $EndComp
@@
 L power:+5V #PWR0106
 U 1 1 5FF5BF4D
-P 10000 2100
-F 0 "#PWR0106" H 10000 1950 50  0001 C CNN
-F 1 "+5V" H 10015 2273 50  0000 C CNN
-F 2 "" H 10000 2100 50  0001 C CNN
-F 3 "" H 10000 2100 50  0001 C CNN
-	1    10000 2100
+P 9350 2200
+F 0 "#PWR0106" H 9350 2050 50  0001 C CNN
+F 1 "+5V" H 9365 2373 50  0000 C CNN
+F 2 "" H 9350 2200 50  0001 C CNN
+F 3 "" H 9350 2200 50  0001 C CNN
+	1    9350 2200
 	1    0    0    -1
 $EndComp
@@
 L power:+5V #PWR0107
 U 1 1 5FF5C6BC
-P 11000 2100
-F 0 "#PWR0107" H 11000 1950 50  0001 C CNN
-F 1 "+5V" H 11015 2273 50  0000 C CNN
-F 2 "" H 11000 2100 50  0001 C CNN
-F 3 "" H 11000 2100 50  0001 C CNN
-	1    11000 2100
+P 10350 2200
+F 0 "#PWR0107" H 10350 2050 50  0001 C CNN
+F 1 "+5V" H 10365 2373 50  0000 C CNN
+F 2 "" H 10350 2200 50  0001 C CNN
+F 3 "" H 10350 2200 50  0001 C CNN
+	1    10350 2200
 	1    0    0    -1
 $EndComp
@@
 $Comp
 L Comparator:LM393 U1
-U 1 1 5FF7CA5E
-P 6000 2450
-F 0 "U1" H 6000 2083 50  0000 C CNN
-F 1 "LM393" H 6000 2174 50  0000 C CNN
-F 2 "Package_SO:SOIC-8_3.9x4.9mm_P1.27mm" H 6000 2450 50  0001 C CNN
-F 3 "http://www.ti.com/lit/ds/symlink/lm393.pdf" H 6000 2450 50  0001 C CNN
-F 4 "C7955" H 6000 2450 50  0001 C CNN "LCSC"
-	1    6000 2450
-	1    0    0    1
-$EndComp
-$Comp
-L Comparator:LM393 U1
 U 2 1 5FF885E6
 P 6000 3100
-F 0 "U1" H 6000 3467 50  0000 C CNN
-F 1 "LM393" H 6000 3376 50  0000 C CNN
+F 0 "U1" H 5950 3100 50  0000 C CNN
+F 1 "MAX9142" H 6000 3376 50  0001 C CNN
 F 2 "Package_SO:SOIC-8_3.9x4.9mm_P1.27mm" H 6000 3100 50  0001 C CNN
 F 3 "http://www.ti.com/lit/ds/symlink/lm393.pdf" H 6000 3100 50  0001 C CNN
@@
 P 10100 1150
 F 0 "U1" H 10058 1196 50  0000 L CNN
-F 1 "LM393" H 10058 1105 50  0000 L CNN
+F 1 "MAX9142" H 10058 1105 50  0000 L CNN
 F 2 "Package_SO:SOIC-8_3.9x4.9mm_P1.27mm" H 10100 1150 50  0001 C CNN
 F 3 "http://www.ti.com/lit/ds/symlink/lm393.pdf" H 10100 1150 50  0001 C CNN
@@
 L Analog_Switch:NC7SB3157P6X U2
 U 2 1 5FF8B772
-P 10000 2600
-F 0 "U2" H 9820 2646 50  0000 R CNN
-F 1 "NC7SB3157P6X" H 9820 2555 50  0000 R CNN
-F 2 "Package_TO_SOT_SMD:SOT-363_SC-70-6" H 10000 2300 50  0001 C CNN
-F 3 "https://www.onsemi.com/pub/Collateral/NC7SB3157-D.PDF" H 10000 2600 50  0001 C CNN
-F 4 "C87403" H 10000 2600 50  0001 C CNN "LCSC"
-	2    10000 2600
+P 9350 2700
+F 0 "U2" H 9170 2746 50  0000 R CNN
+F 1 "NC7SB3157P6X" H 9170 2655 50  0000 R CNN
+F 2 "Package_TO_SOT_SMD:SOT-363_SC-70-6" H 9350 2400 50  0001 C CNN
+F 3 "https://www.onsemi.com/pub/Collateral/NC7SB3157-D.PDF" H 9350 2700 50  0001 C CNN
+F 4 "C87403" H 9350 2700 50  0001 C CNN "LCSC"
+	2    9350 2700
 	-1   0    0    -1
 $EndComp
@@
 L Analog_Switch:NC7SB3157P6X U4
 U 2 1 5FF8FBDB
-P 11000 2600
-F 0 "U4" H 11180 2646 50  0000 L CNN
-F 1 "NC7SB3157P6X" H 11180 2555 50  0000 L CNN
-F 2 "Package_TO_SOT_SMD:SOT-363_SC-70-6" H 11000 2300 50  0001 C CNN
-F 3 "https://www.onsemi.com/pub/Collateral/NC7SB3157-D.PDF" H 11000 2600 50  0001 C CNN
-F 4 "C87403" H 11000 2600 50  0001 C CNN "LCSC"
-	2    11000 2600
+P 10350 2700
+F 0 "U4" H 10530 2746 50  0000 L CNN
+F 1 "NC7SB3157P6X" H 10530 2655 50  0000 L CNN
+F 2 "Package_TO_SOT_SMD:SOT-363_SC-70-6" H 10350 2400 50  0001 C CNN
+F 3 "https://www.onsemi.com/pub/Collateral/NC7SB3157-D.PDF" H 10350 2700 50  0001 C CNN
+F 4 "C87403" H 10350 2700 50  0001 C CNN "LCSC"
+	2    10350 2700
 	1    0    0    -1
 $EndComp
@@
 Text Notes 10200 3700 0    50   ~ 0
 Unused gates
+$Comp
+L Comparator:LM393 U1
+U 1 1 5FF7CA5E
+P 6000 2450
+F 0 "U1" H 5950 2450 50  0000 C CNN
+F 1 "MAX9142" H 6000 2174 50  0001 C CNN
+F 2 "Package_SO:SOIC-8_3.9x4.9mm_P1.27mm" H 6000 2450 50  0001 C CNN
+F 3 "http://www.ti.com/lit/ds/symlink/lm393.pdf" H 6000 2450 50  0001 C CNN
+F 4 "C18567" H 6000 2450 50  0001 C CNN "LCSC"
+	1    6000 2450
+	1    0    0    1
+$EndComp
 $EndSCHEMATC

Commit message: I heard we like LEDs
Parts:
- added D?: LED, LED_SMD:LED_0603_1608Metric, symbol Device:LED
- added R?: 2.2k, Resistor_SMD:R_0402_1005Metric, symbol Device:R
- U1: LCSC C7955 -> C18567
Connections:
- net GND: now also R?.1
- net output: now also D?.2 (A)
- new net: D?.1 (K), R?.2
Changed lines of the file:
@@
 F 2 "Package_SO:SOIC-8_3.9x4.9mm_P1.27mm" H 6000 3100 50  0001 C CNN
 F 3 "http://www.ti.com/lit/ds/symlink/lm393.pdf" H 6000 3100 50  0001 C CNN
-F 4 "C7955" H 6000 3100 50  0001 C CNN "LCSC"
+F 4 "C18567" H 6000 3100 50  0001 C CNN "LCSC"
 	2    6000 3100
 	1    0    0    -1
@@
 F 2 "Package_SO:SOIC-8_3.9x4.9mm_P1.27mm" H 10100 1150 50  0001 C CNN
 F 3 "http://www.ti.com/lit/ds/symlink/lm393.pdf" H 10100 1150 50  0001 C CNN
-F 4 "C7955" H 10100 1150 50  0001 C CNN "LCSC"
+F 4 "C18567" H 10100 1150 50  0001 C CNN "LCSC"
 	3    10100 1150
 	1    0    0    -1
@@
 	1    0    0    1
 $EndComp
+$Comp
+L Device:LED D?
+U 1 1 6049E030
+P 6000 5800
+F 0 "D?" V 6039 5682 50  0000 R CNN
+F 1 "LED" V 5948 5682 50  0000 R CNN
+F 2 "LED_SMD:LED_0603_1608Metric" H 6000 5800 50  0001 C CNN
+F 3 "~" H 6000 5800 50  0001 C CNN
+F 4 "C72043" H 6000 5800 50  0001 C CNN "LCSC"
+	1    6000 5800
+	0    -1   -1   0
+$EndComp
+$Comp
+L Device:R R?
+U 1 1 604A8C15
+P 6000 6100
+F 0 "R?" H 6070 6146 50  0000 L CNN
+F 1 "2.2k" H 6070 6055 50  0000 L CNN
+F 2 "Resistor_SMD:R_0402_1005Metric" V 5930 6100 50  0001 C CNN
+F 3 "~" H 6000 6100 50  0001 C CNN
+F 4 "C25879" H 6000 6100 50  0001 C CNN "LCSC"
+	1    6000 6100
+	1    0    0    1
+$EndComp
+$Comp
+L power:GND #PWR?
+U 1 1 604A981F
+P 6000 6250
+F 0 "#PWR?" H 6000 6000 50  0001 C CNN
+F 1 "GND" H 6005 6077 50  0001 C CNN
+F 2 "" H 6000 6250 50  0001 C CNN
+F 3 "" H 6000 6250 50  0001 C CNN
+	1    6000 6250
+	-1   0    0    -1
+$EndComp
+Text GLabel 5900 5550 0    50   Input ~ 0
+output
+Wire Wire Line
+	5900 5550 6000 5550
+Wire Wire Line
+	6000 5550 6000 5650
 $EndSCHEMATC
